File: GD32F427RE-LTC-SMPTE-no-PHY.kicad_sch (KiCad schematic)
At the start: 64 parts, among them J1 BOOT0, J10 GPS, J11 GPIO 5V, J2 USART0, J3 GPIO, J4 I2C, J5 I2C LCD/KEYS, J6 External PHY, J7 MIDI, J8 SPI, J9 LTC, SW1 BOOT0, SW2 RESET, U1 GT-USB-7010ASV, U2 AMS1117-3.3, U3 W25Q128JVS, U4 74LVC2G125, U5 74LVC2G125, U6 GD32F427RET6, X1 25Mhz, X2 32.768kHz

Commit message: Fix PA3-PA5 pin labels
Correct the PA3, PA4, and PA5 labels in the schematic and PCB silkscreen so the header pin names match the intended mapping. The 3D board render is updated to reflect the corrected labeling.
Connections:
- net PA6 is gone; now on net PA5: J3.4 (Pin_4), U6.21 (PA5)
- net PA4: now also J3.3 (Pin_3), U6.20 (PA4); no longer J3.2 (Pin_2), U6.17 (PA3)
- net PA5: no longer J3.3 (Pin_3), U6.20 (PA4)
- new net PA3: J3.2 (Pin_2), U6.17 (PA3)
Changed lines of the file:
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@@
 		)
 	)
-	(label "PA6"
+	(label "PA5"
 		(at 17.78 77.47 0)
 		(effects
@@
 		)
 	)
-	(label "PA4"
+	(label "PA3"
 		(at 212.09 29.21 0)
 		(effects
@@
 		)
 	)
-	(label "PA6"
+	(label "PA5"
 		(at 212.09 34.29 0)
 		(effects
@@
 		)
 	)
-	(label "PA4"
+	(label "PA3"
 		(at 17.78 82.55 0)
 		(effects
@@
 		)
 	)
-	(label "PA5"
+	(label "PA4"
 		(at 17.78 80.01 0)
 		(effects
@@
 		)
 	)
-	(label "PA5"
+	(label "PA4"
 		(at 212.09 31.75 0)
 		(effects
